File: CL70_PCB.kicad_sch (KiCad schematic)
At the start: 204 parts, among them J1 AVR-ISP-6, SW1 SW_Push, U1 ATmega32U4-MU, U2 PRTR5V0U2X, Y1 16MHz

Commit message: Add wiring
Parts:
- RLED1, RLED2, RLED3: value 1k -> 330
Connections:
- net COL7: now also S47.1
- net COL8: no longer S47.1
- net RESW_A: now also RC5.2; no longer RC4.2
- net RESW_B: now also RC4.2; no longer RC5.2
- net ROW2: now also U1.28 (PB4); no longer U1.29 (PB5)
- net ROW3: now also U1.29 (PB5); no longer U1.28 (PB4)
- net ROW4: now also U1.26 (PD6); no longer U1.27 (PD7)
- net ROW5: now also U1.27 (PD7); no longer U1.26 (PD6)
- net ROW7: now also U1.18 (PD0); no longer U1.22 (PD5)
- net ROW9: now also U1.22 (PD5); no longer U1.20 (PD2)
- net at RC4.1: now also U1.20 (PD2); no longer U1.18 (PD0)
Other:
- moved on the sheet: D47, RC4, S47

Commit message: Add production files
Parts:
- RC1, RC2: value 22k -> 22
Changed lines of the file:
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@@
 			)
 		)
-		(property "Value" "22k"
-			(at 80.264 36.83 90)
+		(property "Value" "22"
+			(at 80.518 36.83 90)
 			(effects
 				(font
@@
 			)
 		)
-		(property "Value" "22k"
-			(at 83.82 46.99 90)
+		(property "Value" "22"
+			(at 83.312 46.99 90)
 			(effects
 				(font
@@
 		)
 		(property "Value" "330"
-			(at 52.07 227.33 90)
+			(at 52.832 227.33 90)
 			(effects
 				(font
@@
 		)
 		(property "Value" "330"
-			(at 52.07 250.19 90)
+			(at 52.832 250.19 90)
 			(effects
 				(font
@@
 		)
 		(property "Value" "330"
-			(at 52.07 238.76 90)
+			(at 52.832 238.76 90)
 			(effects
 				(font
